File: 6500_board/pcg6500.kicad_pcb (KiCad board)
At the start: 2 copper layers, 160 x 138.4 mm, 45 parts, among them CN1 CharROM ADAPTER, CN2 USERPORT, IC1 74LS123, IC10 74LS157, IC11 74LS157, IC12 D2101AL-4, IC13 D2101AL-4, IC14 D2101AL-4, IC15 D2101AL-4, IC2 74LS42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

Commit message: housekeeping
added missing Cap values
improvements in signal naming and schematic layout
no functional changes
Parts:
- C20, C21, C22, C23, C24, C25, C26: value 100nF -> 10nF
- C4: value C_Polarized -> 100uF
- R1: value 10 -> 10R
Connections:
- net /~{WRITE_{RAM}}_{_delayed} renamed /~{WRITE_{RAM}}_{_delay}

Commit message: BOM adjustment
- changed excessive voltage rating of  audio related capacitors to more realistic values
- added cn2 connector to bom
Parts:
- C4: value 100uF -> 100uF 16V
- C5: value 47nF 100V -> 47nF 16V
Changed lines of the file:
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@@
 			)
 		)
-		(property "Value" "47nF 100V"
+		(property "Value" "47nF 16V"
 			(at 3.175 2.2 90)
 			(layer "F.Fab")
@@
 			)
 		)
-		(property "Value" "100uF"
+		(property "Value" "100uF 16V"
 			(at 2.5 5.25 0)
 			(layer "F.Fab")
@@
 		(sheetname "Root")
 		(sheetfile "pcg6500.kicad_sch")
-		(attr through_hole exclude_from_bom)
+		(attr through_hole)
 		(fp_line
 			(start -1.8 24.65)
